File: Schematic & PCB files/moonclock.brd (EAGLE design)
At the start: 145 x 38.4 mm, 27 parts, among them U1 TCA9548APWR, U2 ESP32-S2-WROVER-I, U3 AMS1117-3.3, X2 BM04B-SRSS-TB

Commit message: Updated EAGLE files
Parts:
- moved C6 17.6 mm to (43.3, 8.90), turned to 90 degrees
- moved C5 16.6 mm to (45.4, 8.87), turned to 270 degrees
- moved C4 14.4 mm to (47.6, 8.86), turned to 270 degrees
- moved C7 13.4 mm to (41.0, 8.89), turned to 90 degrees
- moved R2 13.4 mm to (69.8, 11.1)
- moved R1 12.0 mm to (67.4, 11.2), turned to 90 degrees
- moved R4 9.63 mm to (70.2, 20.0), turned to 90 degrees
- moved C3 8.62 mm to (49.8, 8.84), turned to 270 degrees
- moved C2 4.16 mm to (51.9, 8.84), turned to 270 degrees
- moved C1 3.79 mm to (77.1, 22.5), turned to 270 degrees
- moved R3 2.86 mm to (66.4, 20.2), turned to 90 degrees
- moved R6 1.52 mm to (74.9, 22.5), turned to 270 degrees
Connections:
- new net AGND: U2.7
Routing:
- net GND: track 673.1 -> 49.6 mm, vias 8 -> 17
- net AGND: track 0.00 -> 244.3 mm, vias 0 -> 4
- net 0SDA: track 64.3 -> 262.9 mm, vias 4 -> 0
- net VCC: track 225.2 -> 326.3 mm, vias 6 -> 2
- net N$10: track 60.8 -> 129.6 mm
- net INPUTSDA: track 26.6 -> 88.3 mm, vias 3 -> 2
- net N$7: track 130.9 -> 91.7 mm, vias 6 -> 2
- net 0SCL: track 91.1 -> 61.7 mm, vias 1 -> 2
- net RESET: track 11.8 -> 37.3 mm, vias 2 -> 0
- net 1SCL: track 58.1 -> 39.8 mm, vias 3 -> 0
- net 3SCL: track 48.7 -> 38.1 mm, vias 1 -> 0
- net N$6: track 30.5 -> 38.2 mm
- net 4SDA: track 64.7 -> 72.3 mm
- net D-: track 83.8 -> 90.4 mm, vias 0 -> 2
- net 2SDA: track 20.7 -> 27.1 mm, vias 1 -> 0
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- added copper zone on layer 16, net GND

Commit message: PCB
feat: MoonClock add schematics and pcb files
Parts:
- removed U1: TCA9548APWR, microbuilder:TSSOP24
- added C8, C9: 22pF, rcl:C0805
- added D1, D2, D3: CPDQ5V0-HF, CPDQ5V0-HF:MBTB-D-SOD-923F-IMP-0402
- added U4: XC6220B331PR-G, tribonix:SOT-89-5_TOR
- C4: value 22uF -> 0.1uF
- U3: value AMS1117-3.3 -> PCA9547BS,118; device AMS1117-3.3:SOT229P700X180-4N -> PCA9547BS_118:QFN50P400X400X100-25N
- moved U3 32.8 mm to (76.4, 18.5), turned to 180 degrees
- moved C2 27.8 mm to (27.4, 22.0), turned to 180 degrees
- moved C3 24.2 mm to (27.4, 17.9), turned to 180 degrees
- moved C4 23.0 mm to (27.4, 19.9), turned to 180 degrees
- moved C5 19.3 mm to (27.4, 15.9), turned to 180 degrees
- moved C6 17.1 mm to (56.2, 20.2), turned to 0 degrees
- moved C7 16.2 mm to (56.3, 14.1), turned to 0 degrees
- moved R2 11.5 mm to (66.1, 22.0), turned to 180 degrees
- moved R6 9.35 mm to (67.2, 17.2), turned to 180 degrees
- moved R4 9.05 mm to (67.2, 11.5), turned to 0 degrees
- moved C1 8.99 mm to (76.3, 13.6), turned to 0 degrees
- moved R1 8.88 mm to (66.1, 19.9), turned to 180 degrees
- moved R3 6.83 mm to (67.2, 13.4), turned to 0 degrees
- moved BOOT 4.27 mm to (56.3, 23.2)
- moved RESET 4.27 mm to (56.5, 11.0)
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Connections:
- removed net 0SCL: OLED0.2, U1.5
- removed net 0SDA: OLED0.1, U1.4
- removed net 1SCL: OLED1.2, U1.7
- removed net 1SDA: OLED1.1, U1.6
- removed net 2SCL: OLED2.2, U1.9
- removed net 2SDA: OLED2.1, U1.8
- removed net 3SCL: OLED3.2, U1.11
- removed net 3SDA: OLED3.1, U1.10
- removed net 4SCL: OLED4.2, U1.14
- removed net 4SDA: OLED4.1, U1.13
- removed net INPUTSCL: R2.1, U1.22, U2.14
- removed net INPUTSDA: R1.1, U1.23, U2.13
- new net +3V3: C3.1, C5.1, R3.2, R4.2, U4.5
- new net N$1: U2.2
- new net N$11: OLED3.1, U3.7
- new net N$12: OLED4.1, U3.10
- new net N$13: OLED0.2, U3.2
- new net N$14: OLED1.2, U3.4
- new net N$15: OLED2.2, U3.6
- new net N$16: OLED3.2, U3.8
- new net N$17: OLED4.2, U3.11
- new net N$2: R1.1, U2.13, U3.20
- new net N$3: R2.1, U2.14, U3.19
- new net N$4: OLED0.1, U3.1
- new net N$9: OLED2.1, U3.5
- net D+: now also C8.1, D1.2
- net D-: now also C9.1, D2.2
- net GND: now also C8.2, C9.2, D1.1, D2.1, D3.1, U3.9, U4.2; no longer U1.12, U3.1
- net N$7: now also OLED1.1, U3.3; no longer C3.1, C4.1, C5.1, R3.2, R4.2, U2.2, U3.2
- net RESET: now also U3.24; no longer U1.3
- net VCC: now also C4.1, D3.2, U3.21, U4.1, U4.4; no longer U1.24, U3.3
Routing:
- net 0SDA: track 262.9 -> 0.00 mm
- net INPUTSDA: track 88.3 -> 0.00 mm, vias 2 -> 0
- net N$17: track 0.00 -> 74.3 mm
- net 4SCL: track 72.4 -> 0.00 mm
- net 4SDA: track 72.3 -> 0.00 mm
- net N$3: track 0.00 -> 69.8 mm
- net N$10: track 129.6 -> 60.0 mm
- net N$13: track 0.00 -> 66.1 mm
- net N$12: track 0.00 -> 65.4 mm
- net N$2: track 0.00 -> 65.1 mm
- net 0SCL: track 61.7 -> 0.00 mm, vias 2 -> 0
- net N$4: track 0.00 -> 60.9 mm
- net N$7: track 91.7 -> 33.4 mm, vias 2 -> 0
- net +3V3: track 0.00 -> 50.9 mm
- net N$11: track 0.00 -> 44.6 mm
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