File: Schematic & PCB files/usb_board.brd (EAGLE design)
At the start: 145 x 38.4 mm, 2 parts, among them J1 USB4115-03-C_REVA, X1 BM04B-SRSS-TB

Commit message: Updated EAGLE files
Routing:
- net GND: track 436.1 -> 17.5 mm
- net AGND: track 0.00 -> 234.0 mm, vias 0 -> 4
- net VCC: track 39.3 -> 21.6 mm
- net D-: track 24.7 -> 37.8 mm, vias 2 -> 1
- net D+: track 27.6 -> 31.2 mm, vias 1 -> 3
- added copper zone on layer 16, net GND

Commit message: PCB
feat: MoonClock add schematics and pcb files
Parts:
- added D1: MBR0520LT1G, Diode:SODFL3718X115
- added R1, R2: 5.1k, rcl:R0805
- moved X1 3.98 mm to (73.3, 23.9), flipped to the top, turned to 180 degrees
Connections:
- new net N$1: D1.1, X1.1
- new net N$2: J1.A5, R1.2
- new net N$4: J1.B5, R2.2
- net GND: now also R1.1, R2.1
- net VCC: now also D1.2; no longer X1.1
Routing:
- net AGND: track 234.0 -> 0.00 mm, vias 4 -> 1
- net N$2: track 0.00 -> 25.4 mm, vias 0 -> 2
- net D-: track 37.8 -> 17.7 mm, vias 1 -> 0
- net N$4: track 0.00 -> 19.8 mm, vias 0 -> 2
- net D+: track 31.2 -> 22.5 mm
- net N$1: track 0.00 -> 6.23 mm
- net VCC: track 21.6 -> 19.0 mm, vias 1 -> 0
- net GND: track 17.5 -> 19.7 mm, vias 4 -> 6
- net N$6: track 0.00 -> 0.11 mm, vias 0 -> 1
