File: Schematic & PCB files/usb_board.sch (EAGLE design)
At the start: 2 parts, among them J1 USB4115-03-C_REVA, X1 BM04B-SRSS-TB

Commit message: PCB
feat: MoonClock add schematics and pcb files
Parts:
- added D1: MBR0520LT1G, Diode:SCHOTTKY_MBR0520LT1GDO-219
- added R1, R2: 5.1k, rcl:R-EU_R0805
Connections:
- new net N$1: D1.C, X1.1
- new net N$2: J1.CC1, R1.2
- new net N$4: J1.CC2, R2.2
- net GND: now also R1.1, R2.1
- net VCC: now also D1.A; no longer X1.1
